File: HW4/HW4.brd (EAGLE design)
At the start: 100 x 80 mm, 8 parts

Commit message: Finish library + schematic
Parts:
- added LED1, LED2: (no value), HW4:LED3MM
- added R1, R2, R3, R4: (no value), HW4:0207/7
- added U$11: USBUART, HW4:USBUART
- added U$12: DISPLAY, HW4:DISPLAY
- added U$13, U$14, U$6, U$7: ONE, HW4:ONE
- added U$15, U$16, U$17, U$18: FIVE, HW4:FIVE
- added U$19, U$20: PUSH, HW4:PUSH
- added U$9: SLIDE, HW4:SLIDE
- U$2: value SLIDE -> BATTERY; device HW4:SLIDE -> HW4:BATTERY
- U$3: value PUSH -> SNAP; device HW4:PUSH -> HW4:SNAP
- U$4: value PUSH -> VREG; device HW4:PUSH -> HW4:VREG
- U$5: value MICROUSB -> ONE; device HW4:MICROUSB -> HW4:ONE
- moved C1 107.3 mm to (34.3, 29.2), turned to 180 degrees
- moved C2 103.3 mm to (24.1, 53.3)
- moved C3 95.2 mm to (17.8, 35.6)
- moved U$1 93.2 mm to (52.1, 47.0), turned to 270 degrees
- moved U$3 57.3 mm to (7.62, -31.8)
- moved U$4 46.6 mm to (-6.35, -30.5)
- moved U$2 44.7 mm to (-8.89, -83.8)
- moved U$5 42.7 mm to (-10.2, -88.9)
Connections:
- new net +5V: U$9.3, U$9.4
- new net N$1: U$3.1
- new net N$10: U$11.2
- new net N$11: U$11.1
- new net N$12: LED1.K, R4.1
- new net N$13: LED2.K, R3.1
- new net N$14: U$2.2, U$9.1, U$9.6
- new net N$16: U$4.3, U$9.2, U$9.5
- new net N$2: U$3.2
- new net N$3: U$3.3
- new net N$4: U$3.4
- new net N$5: U$3.5
- new net N$6: U$11.6
- new net N$7: U$11.4
- new net N$8: U$11.3
- new net VIN: U$16.2, U$17.1, U$5.P$1
- net +3V3: now also LED1.A, R1.1, R2.1, U$12.2, U$16.1, U$17.4, U$4.1, U$7.P$1
- net A0: now also U$15.3
- net A1: now also U$15.2
- net A3: now also U$15.4
- net A4: now also LED2.A
- net B10: now also U$17.3
- net B11: now also U$18.5
- net B12: now also U$18.4
- net B13: now also U$18.1
- net B14: now also U$18.2
- net B15: now also U$18.3
- net B2: now also U$15.1
- net B4: now also R1.2, U$19.2
- net B5: now also U$15.5
- net B6: now also U$16.3
- net B7: now also U$17.2
- net GND: now also R3.2, R4.2, U$12.1, U$16.4, U$16.5, U$17.5, U$19.1, U$2.1, U$20.1, U$4.2, U$6.P$1
- net MCLR: now also R2.2, U$20.2
- net SCL: now also U$12.3, U$14.P$1
- net SDA: now also U$12.4, U$13.P$1
Other:
- board size 100 x 80 mm -> 100 x 100 mm

Commit message: Board attempt, awful
Parts:
- moved LED2 176.3 mm to (10.2, 47.0), turned to 180 degrees
- moved LED1 172.0 mm to (39.4, 47.0)
- moved R3 164.8 mm to (11.4, 39.4), turned to 270 degrees
- moved R4 160.7 mm to (40.6, 39.4), turned to 270 degrees
- moved R2 150.2 mm to (38.1, 39.4), turned to 90 degrees
- moved R1 139.3 mm to (8.89, 39.4), turned to 90 degrees
- moved U$20 136.6 mm to (45.7, 47.0)
- moved U$19 119.8 mm to (4.19, 46.9)
- moved U$6 113.6 mm to (40.6, 10.2)
- moved U$18 111.9 mm to (47.0, 31.8), turned to 270 degrees
- moved U$7 111.3 mm to (40.6, 5.08)
- moved U$5 104.4 mm to (7.62, 14.0)
- moved U$17 98.7 mm to (47.0, 19.1), turned to 270 degrees
- moved U$2 93.6 mm to (24.1, 3.81), turned to 90 degrees
- moved U$15 91.8 mm to (2.54, 31.8), turned to 270 degrees
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Connections:
- net N$7 renamed U1RX
- removed net N$1: U$3.1
- removed net N$11: U$11.1
- removed net N$2: U$3.2
- removed net N$3: U$3.3
- removed net N$4: U$3.4
- removed net N$5: U$3.5
- removed net N$8: U$11.3
- net +3V3: now also U$16.3, U$3.2; no longer U$16.1
- net +5V: now also U$11.3
- net A0: now also U$15.1; no longer U$15.3
- net B10: now also U$17.1; no longer U$17.3
- net B13: now also U$18.3; no longer U$18.1
- net B15: now also U$18.1; no longer U$18.3
- net B2: now also U$15.3; no longer U$15.1
- net B6: now also U$16.1; no longer U$16.3
- net GND: now also U$11.1, U$3.3
- net MCLR: now also U$3.1
- net PGC: now also U$3.5
- net PGD: now also U$3.4
- net U1TX: now also U$11.5
- net VIN: now also U$17.3; no longer U$17.1
Routing:
- added copper zone on layer 16, net GND
Other:
- board size 100 x 100 mm -> 50 x 50 mm

Commit message: hw4 board/schematic update (finish)
Parts:
- removed LED1: (no value), HW4:LED3MM
- removed R4: (no value), HW4:0207/7
- removed U$3: SNAP, HW4:SNAP
- added LED3: (no value), HW4:LED3MM
- added R5: (no value), HW4:0207/7
- added U$8: USBUART, HW4:USBUART
- C1: value (none) -> 10uF
- C2: value (none) -> 0.1uF; device HW4:C025-030X050 -> HW4:B45181B
- C3: value (none) -> 0.1uF
- U$11: value USBUART -> SNAP; device HW4:USBUART -> HW4:SNAP
- moved U$11 45.3 mm to (25.4, 47.0), turned to 0 degrees
- moved U$5 37.2 mm to (44.5, 19.1)
- moved C3 20.4 mm to (35.6, 41.9)
- moved C1 19.1 mm to (34.3, 21.6), turned to 0 degrees
- moved U$7 12.0 mm to (44.5, 16.5)
- moved U$14 9.92 mm to (33.0, 14.0)
- moved U$4 9.41 mm to (2.03, 5.84), turned to 270 degrees
- moved U$2 8.90 mm to (15.2, 3.43)
- moved R2 8.52 mm to (41.9, 31.8)
- moved U$6 7.62 mm to (40.6, 2.54)
- moved U$9 7.15 mm to (10.9, 5.84), turned to 270 degrees
- moved LED2 7.09 mm to (15.1, 41.9)
- moved U$13 6.84 mm to (33.0, 16.5)
- moved R3 5.74 mm to (13.8, 34.2)
- moved R1 5.22 mm to (9.27, 34.2), turned to 270 degrees
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- renumbered U$15 to U$10, U$16 to U$21
Connections:
- removed net N$10: U$11.2
- removed net N$12: LED1.K, R4.1
- removed net N$6: U$11.6
- new net N$1: C2.+, U$1.13
- new net N$2: LED3.K, R5.1
- net +3V3: now also LED3.A, U$11.2; no longer C2.1, LED1.A, U$1.13, U$3.2
- net +5V: now also U$8.3; no longer U$11.3
- net A0: now also U$10.5; no longer U$10.1
- net A1: now also U$10.4; no longer U$10.2
- net A3: now also U$10.2; no longer U$10.4
- net B5: now also U$10.1; no longer U$10.5
- net B6: now also U$21.5; no longer U$21.1
- net GND: now also C2.-, R5.2, U$11.3, U$21.1, U$21.2, U$8.1; no longer C2.2, R4.2, U$11.1, U$21.4, U$21.5, U$3.3
- net MCLR: now also U$11.1; no longer U$3.1
- net PGC: now also U$11.5; no longer U$3.5
- net PGD: now also U$11.4; no longer U$3.4
- net U1RX: now also U$8.4; no longer U$11.4
- net U1TX: now also U$8.5; no longer U$11.5
- net VIN: now also U$21.4; no longer U$21.2
Routing:
- net +3V3: track 0.00 -> 228.9 mm
- net MCLR: track 0.00 -> 50.7 mm
- net VIN: track 0.00 -> 49.4 mm
- net B4: track 0.00 -> 43.8 mm
- net N$1: track 0.00 -> 40.5 mm
- net U1TX: track 0.00 -> 38.1 mm
- net B6: track 0.00 -> 33.5 mm
- net A4: track 0.00 -> 32.1 mm
- net B5: track 0.00 -> 26.4 mm
- net +5V: track 0.00 -> 25.0 mm
- net PGC: track 0.00 -> 23.4 mm
- net A3: track 0.00 -> 23.3 mm
- net B7: track 0.00 -> 23.0 mm
- net B2: track 0.00 -> 20.1 mm
- net A1: track 0.00 -> 20.1 mm
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