File: HW4/HW4.sch (EAGLE design)
At the start: 8 parts

Commit message: Finish library + schematic
Parts:
- added LED1, LED2: (no value), HW4:LED3MM
- added R1, R2, R3, R4: (no value), HW4:R-US_0207/7
- added U$11: USBUART, HW4:USBUART
- added U$12: DISPLAY, HW4:DISPLAY
- added U$13, U$14, U$6, U$7: ONE, HW4:ONE
- added U$15, U$16, U$17, U$18: FIVE, HW4:FIVE
- added U$19, U$20: PUSH, HW4:PUSH
- added U$9: SLIDE, HW4:SLIDE
- U$2: value SLIDE -> BATTERY; device HW4:SLIDE -> HW4:BATTERY
- U$3: value PUSH -> SNAP; device HW4:PUSH -> HW4:SNAP
- U$4: value PUSH -> VREG; device HW4:PUSH -> HW4:VREG
- U$5: value MICROUSB -> ONE; device HW4:MICROUSB -> HW4:ONE
Connections:
- new net +5V: U$9.3.IN, U$9.4.IN
- new net N$1: U$3.1.MCLR
- new net N$10: U$11.2.CTS
- new net N$11: U$11.1.GND
- new net N$12: LED1.C, R4.1
- new net N$13: LED2.C, R3.1
- new net N$14: U$2.2.VBAT, U$9.1.IN, U$9.6.IN
- new net N$16: U$4.3.VIN, U$9.2.OUT, U$9.5.OUT
- new net N$2: U$3.2.VDD
- new net N$3: U$3.3.GND
- new net N$4: U$3.4.PGD
- new net N$5: U$3.5.PGC
- new net N$6: U$11.6.RTS
- new net N$7: U$11.4.TX
- new net N$8: U$11.3.5V
- new net VIN: U$16.P$2, U$17.P$1, U$5.1
- net +3V3: now also LED1.A, R1.1, R2.1, U$12.2.VCC, U$16.P$1, U$17.P$4, U$4.1.VOUT, U$7.1
- net A0: now also U$15.P$3
- net A1: now also U$15.P$2
- net A3: now also U$15.P$4
- net A4: now also LED2.A
- net B10: now also U$17.P$3
- net B11: now also U$18.P$5
- net B12: now also U$18.P$4
- net B13: now also U$18.P$1
- net B14: now also U$18.P$2
- net B15: now also U$18.P$3
- net B2: now also U$15.P$1
- net B4: now also R1.2, U$19.1
- net B5: now also U$15.P$5
- net B6: now also U$16.P$3
- net B7: now also U$17.P$2
- net GND: now also R3.2, R4.2, U$12.1.GND, U$16.P$4, U$16.P$5, U$17.P$5, U$19.2, U$2.1.GND, U$20.2, U$4.2.GND, U$6.1
- net MCLR: now also R2.2, U$20.1
- net SCL: now also U$12.3.SCL, U$14.1
- net SDA: now also U$12.4.SDA, U$13.1

Commit message: Board attempt, awful
Connections:
- net N$7 renamed U1RX
- removed net N$1: U$3.1.MCLR
- removed net N$11: U$11.1.GND
- removed net N$2: U$3.2.VDD
- removed net N$3: U$3.3.GND
- removed net N$4: U$3.4.PGD
- removed net N$5: U$3.5.PGC
- removed net N$8: U$11.3.5V
- net +3V3: now also U$16.3, U$17.4, U$3.2.VDD; no longer U$16.P$1, U$17.P$4
- net +5V: now also U$11.3.5V
- net A0: now also U$15.1; no longer U$15.P$3
- net A1: now also U$15.2; no longer U$15.P$2
- net A3: now also U$15.4; no longer U$15.P$4
- net B10: now also U$17.1; no longer U$17.P$3
- net B11: now also U$18.5; no longer U$18.P$5
- net B12: now also U$18.4; no longer U$18.P$4
- net B13: now also U$18.3; no longer U$18.P$1
- net B14: now also U$18.2; no longer U$18.P$2
- net B15: now also U$18.1; no longer U$18.P$3
- net B2: now also U$15.3; no longer U$15.P$1
- net B5: now also U$15.5; no longer U$15.P$5
- net B6: now also U$16.1; no longer U$16.P$3
- net B7: now also U$17.2; no longer U$17.P$2
- net GND: now also U$11.1.GND, U$16.4, U$16.5, U$17.5, U$3.3.GND; no longer U$16.P$4, U$16.P$5, U$17.P$5
- net MCLR: now also U$3.1.MCLR
- net PGC: now also U$3.5.PGC
- net PGD: now also U$3.4.PGD
- net U1TX: now also U$11.5.RX
- net VIN: now also U$16.2, U$17.3; no longer U$16.P$2, U$17.P$1

Commit message: hw4 board/schematic update (finish)
Parts:
- removed LED1: (no value), HW4:LED3MM
- removed R4: (no value), HW4:R-US_0207/7
- removed U$15, U$16: FIVE, HW4:FIVE
- removed U$3: SNAP, HW4:SNAP
- added LED3: (no value), HW4:LED3MM
- added R5: (no value), HW4:R-US_0207/7
- added U$10, U$21: FIVE, HW4:FIVE
- added U$8: USBUART, HW4:USBUART
- C1: value (none) -> 10uF
- C2: value (none) -> 0.1uF; device HW4:C-US025-030X050 -> HW4:CPOL-USB45181B
- C3: value (none) -> 0.1uF
- U$11: value USBUART -> SNAP; device HW4:USBUART -> HW4:SNAP
Connections:
- removed net N$10: U$11.2.CTS
- removed net N$12: LED1.C, R4.1
- removed net N$6: U$11.6.RTS
- new net N$1: C2.+, U$1.13.VDD
- new net N$2: LED3.C, R5.1
- net +3V3: now also LED3.A, U$11.2.VDD, U$21.3; no longer C2.1, LED1.A, U$1.13.VDD, U$16.3, U$3.2.VDD
- net +5V: now also U$8.3.5V; no longer U$11.3.5V
- net A0: now also U$10.5; no longer U$15.1
- net A1: now also U$10.4; no longer U$15.2
- net A3: now also U$10.2; no longer U$15.4
- net B2: now also U$10.3; no longer U$15.3
- net B5: now also U$10.1; no longer U$15.5
- net B6: now also U$21.5; no longer U$16.1
- net GND: now also C2.-, R5.2, U$11.3.GND, U$21.1, U$21.2, U$8.1.GND; no longer C2.2, R4.2, U$11.1.GND, U$16.4, U$16.5, U$3.3.GND
- net MCLR: now also U$11.1.MCLR; no longer U$3.1.MCLR
- net PGC: now also U$11.5.PGC; no longer U$3.5.PGC
- net PGD: now also U$11.4.PGD; no longer U$3.4.PGD
- net U1RX: now also U$8.4.TX; no longer U$11.4.TX
- net U1TX: now also U$8.5.RX; no longer U$11.5.RX
- net VIN: now also U$21.4; no longer U$16.2
Other:
- moved on the sheet: LED2, R1, R2, R3, U$12, U$13, U$14, U$17, U$18, U$19, U$2, U$20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
